Commit message: bugs fixed

File: src/my_robot/urdf/my_robot.xacro (robot description, xacro)
@@ -2,5 +2,5 @@
 <robot name="my_robot"
     xmlns:xacro="http://www.ros.org/wiki/xacro">
-    <xacro:include filename="$(find my_robot)/urdf/my_robot.gazebo" />
+    <xacro:include filename="$(find my_robot)/urdf/my_robot.gazebo"/>
     <link name="robot_footprint"></link>
     <link name="chassis">
@@ -103,5 +103,5 @@
         </visual>
     </link>
-    <joint type="continuous" name="left_wheel_hing">
+    <joint type="continuous" name="left_wheel_hinge">
         <origin xyz="0 0.15 0" rpy="0 0 0"/>
         <parent link="chassis"/>
@@ -111,5 +111,5 @@
         <dynamics damping="1.0" friction="1.0"/>
     </joint>
-    <joint type="continuous" name="right_wheel_hing">
+    <joint type="continuous" name="right_wheel_hinge">
         <origin xyz="0 -0.15 0" rpy="0 0 0"/>
         <parent link="chassis"/>

Commit message: updated the structure of the project as requried

File: src/my_robot/urdf/my_robot.xacro (robot description, xacro)
@@ -7,5 +7,5 @@
         <pose>0 0 0.1 0 0 0</pose>
         <inertial>
-            <mass value="15.0"/>
+            <mass value="20.0"/>
             <origin xyz="0 0 0" rpy="0 0 0"/>
             <inertia
@@ -18,5 +18,5 @@
             <origin xyz="0 0 0" rpy="0 0 0"/>
             <geometry>
-                <box size=".4 .2 .1"/>
+                <box size=".4 .4 .2"/>
             </geometry>
         </collision>
@@ -24,29 +24,29 @@
             <origin xyz="0 0 0" rpy="0 0 0"/>
             <geometry>
-                <box size=".4 .2 .1"/>
+                <box size=".4 .4 .2"/>
             </geometry>
         </visual>
         <collision name="back_caster_collision">
-            <origin xyz="-0.15 0 -0.05" rpy="0 0 0"/>
+            <origin xyz="-0.1 0 -0.075" rpy="0 0 0"/>
             <geometry>
-                <sphere radius="0.0499"/>
+                <sphere radius="0.0749"/>
             </geometry>
         </collision>
         <visual name="back_caster_visual">
-            <origin xyz="-0.15 0 -0.05" rpy="0 0 0"/>
+            <origin xyz="-0.1 0 -0.075" rpy="0 0 0"/>
             <geometry>
-                <sphere radius="0.05"/>
+                <sphere radius="0.075"/>
             </geometry>
         </visual>
         <collision name="front_caster_collision">
-            <origin xyz="0.15 0 -0.05" rpy="0 0 0"/>
+            <origin xyz="0.1 0 -0.075" rpy="0 0 0"/>
             <geometry>
-                <sphere radius="0.0499"/>
+                <sphere radius="0.0749"/>
             </geometry>
         </collision>
         <visual name="front_caster_visual">
-            <origin xyz="0.15 0 -0.05" rpy="0 0 0"/>
+            <origin xyz="0.1 0 -0.075" rpy="0 0 0"/>
             <geometry>
-                <sphere radius="0.05"/>
+                <sphere radius="0.075"/>
             </geometry>
         </visual>
@@ -70,5 +70,5 @@
             <origin xyz="0 0 0" rpy="0 1.5707 1.5707"/>
             <geometry>
-                <cylinder radius="0.1" length="0.05"/>
+                <cylinder radius="0.15" length="0.07"/>
             </geometry>
         </collision>
@@ -76,5 +76,5 @@
             <origin xyz="0 0 0" rpy="0 1.5707 1.5707"/>
             <geometry>
-                <cylinder radius="0.1" length="0.05"/>
+                <cylinder radius="0.15" length="0.07"/>
             </geometry>
         </visual>
@@ -93,5 +93,5 @@
             <origin xyz="0 0 0" rpy="0 1.5707 1.5707"/>
             <geometry>
-                <cylinder radius="0.1" length="0.05"/>
+                <cylinder radius="0.15" length="0.07"/>
             </geometry>
         </collision>
@@ -99,10 +99,10 @@
             <origin xyz="0 0 0" rpy="0 1.5707 1.5707"/>
             <geometry>
-                <cylinder radius="0.1" length="0.05"/>
+                <cylinder radius="0.15" length="0.07"/>
             </geometry>
         </visual>
     </link>
     <joint type="continuous" name="left_wheel_hinge">
-        <origin xyz="0 0.15 0" rpy="0 0 0"/>
+        <origin xyz="0 0.25 0" rpy="0 0 0"/>
         <parent link="chassis"/>
         <child link="left_wheel"/>
@@ -112,5 +112,5 @@
     </joint>
     <joint type="continuous" name="right_wheel_hinge">
-        <origin xyz="0 -0.15 0" rpy="0 0 0"/>
+        <origin xyz="0 -0.25 0" rpy="0 0 0"/>
         <parent link="chassis"/>
         <child link="right_wheel"/>
@@ -143,5 +143,5 @@
     </link>
     <joint type="fixed" name="camera_joint">
-        <origin xyz="0.2 0 0" rpy="0 0 0"/>
+        <origin xyz="0.2 0 0.05" rpy="0 0 0"/>
         <parent link="chassis"/>
         <child link="camera"/>
@@ -171,5 +171,5 @@
     </link>
     <joint type="fixed" name="hokuyo_joint">
-        <origin xyz="0.15 0 0.1" rpy="0 0 0"/>
+        <origin xyz="0.15 0 0.15" rpy="0 0 0"/>
         <axis xyz="0 1 0" rpy="0 0 0"/>
         <parent link="chassis"/>
@@ -177,11 +177,11 @@
     </joint>
     <gazebo reference="left_wheel">
-        <material>Gazebo/Green</material>
+        <material>Gazebo/Grey</material>
     </gazebo>
     <gazebo reference="right_wheel">
-        <material>Gazebo/Green</material>
+        <material>Gazebo/Grey</material>
     </gazebo>
     <gazebo reference="chassis">
-        <material>Gazebo/Blue</material>
+        <material>Gazebo/Orange</material>
     </gazebo>
     <gazebo reference="camera">
